File: core/ledchain1.sch (KiCad schematic (older format))
At the start: 60 parts, among them U33 WS2811, U34 WS2811, U35 WS2811, U36 WS2811, U37 WS2811, U38 WS2811, U39 WS2811, U40 WS2811, U41 WS2811, U42 WS2811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

Commit message: Fixed ERC errors and initially populated board
Parts:
- renumbered D103 to D301, D108 to D302, D113 to D303, D118 to D304, D123 to D305, D128 to D306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
