File: core/core.kicad_pcb (KiCad board)
At the start: 2 copper layers, 288 parts, among them K501 KEYSW, K502 KEYSW, K503 KEYSW, K504 KEYSW, K505 KEYSW, K506 KEYSW, K507 KEYSW, K508 KEYSW, K509 KEYSW, K510 KEYSW, K511 KEYSW, K512 KEYSW, K513 KEYSW, K514 KEYSW, K515 KEYSW, K516 KEYSW, K517 KEYSW, K518 KEYSW, K519 KEYSW, K520 KEYSW, K521 KEYSW, K522 KEYSW, K523 KEYSW, K524 KEYSW, K525 KEYSW, K526 KEYSW, K527 KEYSW, K528 KEYSW, K529 KEYSW, K530 KEYSW, K531 KEYSW, K532 KEYSW, K533 KEYSW, K534 KEYSW, K535 KEYSW, K536 KEYSW, K537 KEYSW, K538 KEYSW, K539 KEYSW, K540 KEYSW, K541 KEYSW, K542 KEYSW, K543 KEYSW, K544 KEYSW, K545 KEYSW, K546 KEYSW, K547 KEYSW, K548 KEYSW, K549 KEYSW, K550 KEYSW, K551 KEYSW, K552 KEYSW, K553 KEYSW, K554 KEYSW, K555 KEYSW, K556 KEYSW, K557 KEYSW, K558 KEYSW, K559 KEYSW, K560 KEYSW, K561 KEYSW, K562 KEYSW, K563 KEYSW, K564 KEYSW, K565 KEYSW, K566 KEYSW, K567 KEYSW, K568 KEYSW, K569 KEYSW, K570 KEYSW, K571 KEYSW, K572 KEYSW, U101 Teensy-LC, U201 WS2811, U202 WS2811, U203 WS2811, U204 WS2811, U205 WS2811, U206 WS2811, U207 WS2811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

Commit message: separate footprints on PCB and put some diodes with their keyswitches
Parts:
- moved D507 281.6 mm to (298.2, 68.6)
- moved D509 281.6 mm to (308.6, 72.2)
- moved D510 281.6 mm to (308.6, 68.6)
- moved D512 281.6 mm to (298.2, 72.2)
- moved D514 281.6 mm to (329.4, 68.6)
- moved D515 281.6 mm to (329.4, 72.2)
- moved D520 281.6 mm to (350.2, 68.6)
- moved D508 281.6 mm to (308.6, 75.8)
- moved D511 281.6 mm to (298.2, 75.8)
- moved D517 281.6 mm to (329.4, 75.8)
- moved D518 281.6 mm to (339.8, 68.6)
- moved D519 281.6 mm to (319.0, 68.6)
- moved D525 281.6 mm to (319.0, 72.2)
- moved D516 281.6 mm to (319.0, 75.8)
- moved D526 217.7 mm to (319.5, 92.5)
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