File: test_board/ledchain0.sch (KiCad schematic (older format))
At the start: 32 parts, among them U201 WS2811, U202 WS2811, U203 WS2811, U204 WS2811, U205 WS2811, U206 WS2811, U207 WS2811, U208 WS2811, U209 WS2811, U210 WS2811, U211 WS2811, U212 WS2811, U213 WS2811, U214 WS2811, U215 WS2811, U216 WS2811

Commit message: Updated LED footprints
Parts:
- D201, D202, D203, D204, D205, D206, D207, D208, D209, D210, D211, D212, D213, D214, D215, D216: footprint Connector_PinHeader_1.00mm:PinHeader_1x04_P1.00mm_Horizontal -> LED_THT:LED_D5.0mm-4_RGB
Changed lines of the file:
@@
 F 0 "D205" H 2950 6597 50  0000 C CNN
 F 1 "LED_RCBG" H 2950 6506 50  0000 C CNN
-F 2 "Connector_PinHeader_1.00mm:PinHeader_1x04_P1.00mm_Horizontal" H 2950 6050 50  0001 C CNN
+F 2 "LED_THT:LED_D5.0mm-4_RGB" H 2950 6050 50  0001 C CNN
 F 3 "~" H 2950 6050 50  0001 C CNN
 	1    2950 6100
@@
 F 0 "D204" H 2950 5447 50  0000 C CNN
 F 1 "LED_RCBG" H 2950 5356 50  0000 C CNN
-F 2 "Connector_PinHeader_1.00mm:PinHeader_1x04_P1.00mm_Horizontal" H 2950 4900 50  0001 C CNN
+F 2 "LED_THT:LED_D5.0mm-4_RGB" H 2950 4900 50  0001 C CNN
 F 3 "~" H 2950 4900 50  0001 C CNN
 	1    2950 4950
@@
 F 0 "D203" H 2950 4297 50  0000 C CNN
 F 1 "LED_RCBG" H 2950 4206 50  0000 C CNN
-F 2 "Connector_PinHeader_1.00mm:PinHeader_1x04_P1.00mm_Horizontal" H 2950 3750 50  0001 C CNN
+F 2 "LED_THT:LED_D5.0mm-4_RGB" H 2950 3750 50  0001 C CNN
 F 3 "~" H 2950 3750 50  0001 C CNN
 	1    2950 3800
@@
 F 0 "D202" H 2950 3147 50  0000 C CNN
 F 1 "LED_RCBG" H 2950 3056 50  0000 C CNN
-F 2 "Connector_PinHeader_1.00mm:PinHeader_1x04_P1.00mm_Horizontal" H 2950 2600 50  0001 C CNN
+F 2 "LED_THT:LED_D5.0mm-4_RGB" H 2950 2600 50  0001 C CNN
 F 3 "~" H 2950 2600 50  0001 C CNN
 	1    2950 2650
@@
 F 0 "D201" H 2950 1997 50  0000 C CNN
 F 1 "LED_RCBG" H 2950 1906 50  0000 C CNN
-F 2 "Connector_PinHeader_1.00mm:PinHeader_1x04_P1.00mm_Horizontal" H 2950 1450 50  0001 C CNN
+F 2 "LED_THT:LED_D5.0mm-4_RGB" H 2950 1450 50  0001 C CNN
 F 3 "~" H 2950 1450 50  0001 C CNN
 	1    2950 1500
@@
 F 0 "D210" H 4500 6597 50  0000 C CNN
 F 1 "LED_RCBG" H 4500 6506 50  0000 C CNN
-F 2 "Connector_PinHeader_1.00mm:PinHeader_1x04_P1.00mm_Horizontal" H 4500 6050 50  0001 C CNN
+F 2 "LED_THT:LED_D5.0mm-4_RGB" H 4500 6050 50  0001 C CNN
 F 3 "~" H 4500 6050 50  0001 C CNN
 	1    4500 6100
@@
 F 0 "D209" H 4500 5447 50  0000 C CNN
 F 1 "LED_RCBG" H 4500 5356 50  0000 C CNN
-F 2 "Connector_PinHeader_1.00mm:PinHeader_1x04_P1.00mm_Horizontal" H 4500 4900 50  0001 C CNN
+F 2 "LED_THT:LED_D5.0mm-4_RGB" H 4500 4900 50  0001 C CNN
 F 3 "~" H 4500 4900 50  0001 C CNN
 	1    4500 4950
@@
 F 0 "D208" H 4500 4297 50  0000 C CNN
 F 1 "LED_RCBG" H 4500 4206 50  0000 C CNN
-F 2 "Connector_PinHeader_1.00mm:PinHeader_1x04_P1.00mm_Horizontal" H 4500 3750 50  0001 C CNN
+F 2 "LED_THT:LED_D5.0mm-4_RGB" H 4500 3750 50  0001 C CNN
 F 3 "~" H 4500 3750 50  0001 C CNN
 	1    4500 3800
@@
 F 0 "D207" H 4500 3147 50  0000 C CNN
 F 1 "LED_RCBG" H 4500 3056 50  0000 C CNN
-F 2 "Connector_PinHeader_1.00mm:PinHeader_1x04_P1.00mm_Horizontal" H 4500 2600 50  0001 C CNN
+F 2 "LED_THT:LED_D5.0mm-4_RGB" H 4500 2600 50  0001 C CNN
 F 3 "~" H 4500 2600 50  0001 C CNN
 	1    4500 2650
@@
 F 0 "D206" H 4500 1997 50  0000 C CNN
 F 1 "LED_RCBG" H 4500 1906 50  0000 C CNN
-F 2 "Connector_PinHeader_1.00mm:PinHeader_1x04_P1.00mm_Horizontal" H 4500 1450 50  0001 C CNN
+F 2 "LED_THT:LED_D5.0mm-4_RGB" H 4500 1450 50  0001 C CNN
 F 3 "~" H 4500 1450 50  0001 C CNN
 	1    4500 1500
@@
 F 0 "D215" H 6050 6597 50  0000 C CNN
 F 1 "LED_RCBG" H 6050 6506 50  0000 C CNN
-F 2 "Connector_PinHeader_1.00mm:PinHeader_1x04_P1.00mm_Horizontal" H 6050 6050 50  0001 C CNN
+F 2 "LED_THT:LED_D5.0mm-4_RGB" H 6050 6050 50  0001 C CNN
 F 3 "~" H 6050 6050 50  0001 C CNN
 	1    6050 6100
@@
 F 0 "D214" H 6050 5447 50  0000 C CNN
 F 1 "LED_RCBG" H 6050 5356 50  0000 C CNN
-F 2 "Connector_PinHeader_1.00mm:PinHeader_1x04_P1.00mm_Horizontal" H 6050 4900 50  0001 C CNN
+F 2 "LED_THT:LED_D5.0mm-4_RGB" H 6050 4900 50  0001 C CNN
 F 3 "~" H 6050 4900 50  0001 C CNN
 	1    6050 4950
@@
 F 0 "D213" H 6050 4297 50  0000 C CNN
 F 1 "LED_RCBG" H 6050 4206 50  0000 C CNN
-F 2 "Connector_PinHeader_1.00mm:PinHeader_1x04_P1.00mm_Horizontal" H 6050 3750 50  0001 C CNN
+F 2 "LED_THT:LED_D5.0mm-4_RGB" H 6050 3750 50  0001 C CNN
 F 3 "~" H 6050 3750 50  0001 C CNN
 	1    6050 3800
@@
 F 0 "D212" H 6050 3147 50  0000 C CNN
 F 1 "LED_RCBG" H 6050 3056 50  0000 C CNN
-F 2 "Connector_PinHeader_1.00mm:PinHeader_1x04_P1.00mm_Horizontal" H 6050 2600 50  0001 C CNN
+F 2 "LED_THT:LED_D5.0mm-4_RGB" H 6050 2600 50  0001 C CNN
 F 3 "~" H 6050 2600 50  0001 C CNN
 	1    6050 2650
@@
 F 0 "D211" H 6050 1997 50  0000 C CNN
 F 1 "LED_RCBG" H 6050 1906 50  0000 C CNN
-F 2 "Connector_PinHeader_1.00mm:PinHeader_1x04_P1.00mm_Horizontal" H 6050 1450 50  0001 C CNN
+F 2 "LED_THT:LED_D5.0mm-4_RGB" H 6050 1450 50  0001 C CNN
 F 3 "~" H 6050 1450 50  0001 C CNN
 	1    6050 1500
@@
 F 0 "D216" H 7600 1997 50  0000 C CNN
 F 1 "LED_RCBG" H 7600 1906 50  0000 C CNN
-F 2 "Connector_PinHeader_1.00mm:PinHeader_1x04_P1.00mm_Horizontal" H 7600 1450 50  0001 C CNN
+F 2 "LED_THT:LED_D5.0mm-4_RGB" H 7600 1450 50  0001 C CNN
 F 3 "~" H 7600 1450 50  0001 C CNN
 	1    7600 1500

Commit message: remove through hole leds
Parts:
- D201, D202, D203, D204, D205, D206, D207, D208, D209, D210, D211, D212, D213, D214, D215, D216: footprint LED_THT:LED_D5.0mm-4_RGB -> keyboard_project:NPPN041BFLD-RC
Changed lines of the file:
@@
 F 0 "D205" H 2950 6597 50  0000 C CNN
 F 1 "LED_RCBG" H 2950 6506 50  0000 C CNN
-F 2 "LED_THT:LED_D5.0mm-4_RGB" H 2950 6050 50  0001 C CNN
+F 2 "keyboard_project:NPPN041BFLD-RC" H 2950 6050 50  0001 C CNN
 F 3 "~" H 2950 6050 50  0001 C CNN
 	1    2950 6100
@@
 F 0 "D204" H 2950 5447 50  0000 C CNN
 F 1 "LED_RCBG" H 2950 5356 50  0000 C CNN
-F 2 "LED_THT:LED_D5.0mm-4_RGB" H 2950 4900 50  0001 C CNN
+F 2 "keyboard_project:NPPN041BFLD-RC" H 2950 4900 50  0001 C CNN
 F 3 "~" H 2950 4900 50  0001 C CNN
 	1    2950 4950
@@
 F 0 "D203" H 2950 4297 50  0000 C CNN
 F 1 "LED_RCBG" H 2950 4206 50  0000 C CNN
-F 2 "LED_THT:LED_D5.0mm-4_RGB" H 2950 3750 50  0001 C CNN
+F 2 "keyboard_project:NPPN041BFLD-RC" H 2950 3750 50  0001 C CNN
 F 3 "~" H 2950 3750 50  0001 C CNN
 	1    2950 3800
@@
 F 0 "D202" H 2950 3147 50  0000 C CNN
 F 1 "LED_RCBG" H 2950 3056 50  0000 C CNN
-F 2 "LED_THT:LED_D5.0mm-4_RGB" H 2950 2600 50  0001 C CNN
+F 2 "keyboard_project:NPPN041BFLD-RC" H 2950 2600 50  0001 C CNN
 F 3 "~" H 2950 2600 50  0001 C CNN
 	1    2950 2650
@@
 F 0 "D201" H 2950 1997 50  0000 C CNN
 F 1 "LED_RCBG" H 2950 1906 50  0000 C CNN
-F 2 "LED_THT:LED_D5.0mm-4_RGB" H 2950 1450 50  0001 C CNN
+F 2 "keyboard_project:NPPN041BFLD-RC" H 2950 1450 50  0001 C CNN
 F 3 "~" H 2950 1450 50  0001 C CNN
 	1    2950 1500
@@
 F 0 "D210" H 4500 6597 50  0000 C CNN
 F 1 "LED_RCBG" H 4500 6506 50  0000 C CNN
-F 2 "LED_THT:LED_D5.0mm-4_RGB" H 4500 6050 50  0001 C CNN
+F 2 "keyboard_project:NPPN041BFLD-RC" H 4500 6050 50  0001 C CNN
 F 3 "~" H 4500 6050 50  0001 C CNN
 	1    4500 6100
@@
 F 0 "D209" H 4500 5447 50  0000 C CNN
 F 1 "LED_RCBG" H 4500 5356 50  0000 C CNN
-F 2 "LED_THT:LED_D5.0mm-4_RGB" H 4500 4900 50  0001 C CNN
+F 2 "keyboard_project:NPPN041BFLD-RC" H 4500 4900 50  0001 C CNN
 F 3 "~" H 4500 4900 50  0001 C CNN
 	1    4500 4950
@@
 F 0 "D208" H 4500 4297 50  0000 C CNN
 F 1 "LED_RCBG" H 4500 4206 50  0000 C CNN
-F 2 "LED_THT:LED_D5.0mm-4_RGB" H 4500 3750 50  0001 C CNN
+F 2 "keyboard_project:NPPN041BFLD-RC" H 4500 3750 50  0001 C CNN
 F 3 "~" H 4500 3750 50  0001 C CNN
 	1    4500 3800
@@
 F 0 "D207" H 4500 3147 50  0000 C CNN
 F 1 "LED_RCBG" H 4500 3056 50  0000 C CNN
-F 2 "LED_THT:LED_D5.0mm-4_RGB" H 4500 2600 50  0001 C CNN
+F 2 "keyboard_project:NPPN041BFLD-RC" H 4500 2600 50  0001 C CNN
 F 3 "~" H 4500 2600 50  0001 C CNN
 	1    4500 2650
@@
 F 0 "D206" H 4500 1997 50  0000 C CNN
 F 1 "LED_RCBG" H 4500 1906 50  0000 C CNN
-F 2 "LED_THT:LED_D5.0mm-4_RGB" H 4500 1450 50  0001 C CNN
+F 2 "keyboard_project:NPPN041BFLD-RC" H 4500 1450 50  0001 C CNN
 F 3 "~" H 4500 1450 50  0001 C CNN
 	1    4500 1500
@@
 F 0 "D215" H 6050 6597 50  0000 C CNN
 F 1 "LED_RCBG" H 6050 6506 50  0000 C CNN
-F 2 "LED_THT:LED_D5.0mm-4_RGB" H 6050 6050 50  0001 C CNN
+F 2 "keyboard_project:NPPN041BFLD-RC" H 6050 6050 50  0001 C CNN
 F 3 "~" H 6050 6050 50  0001 C CNN
 	1    6050 6100
@@
 F 0 "D214" H 6050 5447 50  0000 C CNN
 F 1 "LED_RCBG" H 6050 5356 50  0000 C CNN
-F 2 "LED_THT:LED_D5.0mm-4_RGB" H 6050 4900 50  0001 C CNN
+F 2 "keyboard_project:NPPN041BFLD-RC" H 6050 4900 50  0001 C CNN
 F 3 "~" H 6050 4900 50  0001 C CNN
 	1    6050 4950
@@
 F 0 "D213" H 6050 4297 50  0000 C CNN
 F 1 "LED_RCBG" H 6050 4206 50  0000 C CNN
-F 2 "LED_THT:LED_D5.0mm-4_RGB" H 6050 3750 50  0001 C CNN
+F 2 "keyboard_project:NPPN041BFLD-RC" H 6050 3750 50  0001 C CNN
 F 3 "~" H 6050 3750 50  0001 C CNN
 	1    6050 3800
@@
 F 0 "D212" H 6050 3147 50  0000 C CNN
 F 1 "LED_RCBG" H 6050 3056 50  0000 C CNN
-F 2 "LED_THT:LED_D5.0mm-4_RGB" H 6050 2600 50  0001 C CNN
+F 2 "keyboard_project:NPPN041BFLD-RC" H 6050 2600 50  0001 C CNN
 F 3 "~" H 6050 2600 50  0001 C CNN
 	1    6050 2650
@@
 F 0 "D211" H 6050 1997 50  0000 C CNN
 F 1 "LED_RCBG" H 6050 1906 50  0000 C CNN
-F 2 "LED_THT:LED_D5.0mm-4_RGB" H 6050 1450 50  0001 C CNN
+F 2 "keyboard_project:NPPN041BFLD-RC" H 6050 1450 50  0001 C CNN
 F 3 "~" H 6050 1450 50  0001 C CNN
 	1    6050 1500
@@
 F 0 "D216" H 7600 1997 50  0000 C CNN
 F 1 "LED_RCBG" H 7600 1906 50  0000 C CNN
-F 2 "LED_THT:LED_D5.0mm-4_RGB" H 7600 1450 50  0001 C CNN
+F 2 "keyboard_project:NPPN041BFLD-RC" H 7600 1450 50  0001 C CNN
 F 3 "~" H 7600 1450 50  0001 C CNN
 	1    7600 1500

Commit message: update test board schematic to SMD LED
Parts:
- D201, D202, D203, D204, D205, D206, D207, D208, D209, D210, D211, D212, D213, D214, D215, D216: footprint keyboard_project:NPPN041BFLD-RC -> keyboard_project:APTF1616SEJ3ZGGVBDC
Changed lines of the file:
@@
 EESchema Schematic File Version 4
-LIBS:test_board-cache
 EELAYER 30 0
 EELAYER END
@@
 F 0 "D205" H 2950 6597 50  0000 C CNN
 F 1 "LED_RCBG" H 2950 6506 50  0000 C CNN
-F 2 "keyboard_project:NPPN041BFLD-RC" H 2950 6050 50  0001 C CNN
+F 2 "keyboard_project:APTF1616SEJ3ZGGVBDC" H 2950 6050 50  0001 C CNN
 F 3 "~" H 2950 6050 50  0001 C CNN
 	1    2950 6100
@@
 F 0 "D204" H 2950 5447 50  0000 C CNN
 F 1 "LED_RCBG" H 2950 5356 50  0000 C CNN
-F 2 "keyboard_project:NPPN041BFLD-RC" H 2950 4900 50  0001 C CNN
+F 2 "keyboard_project:APTF1616SEJ3ZGGVBDC" H 2950 4900 50  0001 C CNN
 F 3 "~" H 2950 4900 50  0001 C CNN
 	1    2950 4950
@@
 F 0 "D203" H 2950 4297 50  0000 C CNN
 F 1 "LED_RCBG" H 2950 4206 50  0000 C CNN
-F 2 "keyboard_project:NPPN041BFLD-RC" H 2950 3750 50  0001 C CNN
+F 2 "keyboard_project:APTF1616SEJ3ZGGVBDC" H 2950 3750 50  0001 C CNN
 F 3 "~" H 2950 3750 50  0001 C CNN
 	1    2950 3800
@@
 F 0 "D202" H 2950 3147 50  0000 C CNN
 F 1 "LED_RCBG" H 2950 3056 50  0000 C CNN
-F 2 "keyboard_project:NPPN041BFLD-RC" H 2950 2600 50  0001 C CNN
+F 2 "keyboard_project:APTF1616SEJ3ZGGVBDC" H 2950 2600 50  0001 C CNN
 F 3 "~" H 2950 2600 50  0001 C CNN
 	1    2950 2650
@@
 F 0 "D201" H 2950 1997 50  0000 C CNN
 F 1 "LED_RCBG" H 2950 1906 50  0000 C CNN
-F 2 "keyboard_project:NPPN041BFLD-RC" H 2950 1450 50  0001 C CNN
+F 2 "keyboard_project:APTF1616SEJ3ZGGVBDC" H 2950 1450 50  0001 C CNN
 F 3 "~" H 2950 1450 50  0001 C CNN
 	1    2950 1500
@@
 F 0 "D210" H 4500 6597 50  0000 C CNN
 F 1 "LED_RCBG" H 4500 6506 50  0000 C CNN
-F 2 "keyboard_project:NPPN041BFLD-RC" H 4500 6050 50  0001 C CNN
+F 2 "keyboard_project:APTF1616SEJ3ZGGVBDC" H 4500 6050 50  0001 C CNN
 F 3 "~" H 4500 6050 50  0001 C CNN
 	1    4500 6100
@@
 F 0 "D209" H 4500 5447 50  0000 C CNN
 F 1 "LED_RCBG" H 4500 5356 50  0000 C CNN
-F 2 "keyboard_project:NPPN041BFLD-RC" H 4500 4900 50  0001 C CNN
+F 2 "keyboard_project:APTF1616SEJ3ZGGVBDC" H 4500 4900 50  0001 C CNN
 F 3 "~" H 4500 4900 50  0001 C CNN
 	1    4500 4950
@@
 F 0 "D208" H 4500 4297 50  0000 C CNN
 F 1 "LED_RCBG" H 4500 4206 50  0000 C CNN
-F 2 "keyboard_project:NPPN041BFLD-RC" H 4500 3750 50  0001 C CNN
+F 2 "keyboard_project:APTF1616SEJ3ZGGVBDC" H 4500 3750 50  0001 C CNN
 F 3 "~" H 4500 3750 50  0001 C CNN
 	1    4500 3800
@@
 F 0 "D207" H 4500 3147 50  0000 C CNN
 F 1 "LED_RCBG" H 4500 3056 50  0000 C CNN
-F 2 "keyboard_project:NPPN041BFLD-RC" H 4500 2600 50  0001 C CNN
+F 2 "keyboard_project:APTF1616SEJ3ZGGVBDC" H 4500 2600 50  0001 C CNN
 F 3 "~" H 4500 2600 50  0001 C CNN
 	1    4500 2650
@@
 F 0 "D206" H 4500 1997 50  0000 C CNN
 F 1 "LED_RCBG" H 4500 1906 50  0000 C CNN
-F 2 "keyboard_project:NPPN041BFLD-RC" H 4500 1450 50  0001 C CNN
+F 2 "keyboard_project:APTF1616SEJ3ZGGVBDC" H 4500 1450 50  0001 C CNN
 F 3 "~" H 4500 1450 50  0001 C CNN
 	1    4500 1500
@@
 F 0 "D215" H 6050 6597 50  0000 C CNN
 F 1 "LED_RCBG" H 6050 6506 50  0000 C CNN
-F 2 "keyboard_project:NPPN041BFLD-RC" H 6050 6050 50  0001 C CNN
+F 2 "keyboard_project:APTF1616SEJ3ZGGVBDC" H 6050 6050 50  0001 C CNN
 F 3 "~" H 6050 6050 50  0001 C CNN
 	1    6050 6100
@@
 F 0 "D214" H 6050 5447 50  0000 C CNN
 F 1 "LED_RCBG" H 6050 5356 50  0000 C CNN
-F 2 "keyboard_project:NPPN041BFLD-RC" H 6050 4900 50  0001 C CNN
+F 2 "keyboard_project:APTF1616SEJ3ZGGVBDC" H 6050 4900 50  0001 C CNN
 F 3 "~" H 6050 4900 50  0001 C CNN
 	1    6050 4950
@@
 F 0 "D213" H 6050 4297 50  0000 C CNN
 F 1 "LED_RCBG" H 6050 4206 50  0000 C CNN
-F 2 "keyboard_project:NPPN041BFLD-RC" H 6050 3750 50  0001 C CNN
+F 2 "keyboard_project:APTF1616SEJ3ZGGVBDC" H 6050 3750 50  0001 C CNN
 F 3 "~" H 6050 3750 50  0001 C CNN
 	1    6050 3800
@@
 F 0 "D212" H 6050 3147 50  0000 C CNN
 F 1 "LED_RCBG" H 6050 3056 50  0000 C CNN
-F 2 "keyboard_project:NPPN041BFLD-RC" H 6050 2600 50  0001 C CNN
+F 2 "keyboard_project:APTF1616SEJ3ZGGVBDC" H 6050 2600 50  0001 C CNN
 F 3 "~" H 6050 2600 50  0001 C CNN
 	1    6050 2650
@@
 F 0 "D211" H 6050 1997 50  0000 C CNN
 F 1 "LED_RCBG" H 6050 1906 50  0000 C CNN
-F 2 "keyboard_project:NPPN041BFLD-RC" H 6050 1450 50  0001 C CNN
+F 2 "keyboard_project:APTF1616SEJ3ZGGVBDC" H 6050 1450 50  0001 C CNN
 F 3 "~" H 6050 1450 50  0001 C CNN
 	1    6050 1500
@@
 F 0 "D216" H 7600 1997 50  0000 C CNN
 F 1 "LED_RCBG" H 7600 1906 50  0000 C CNN
-F 2 "keyboard_project:NPPN041BFLD-RC" H 7600 1450 50  0001 C CNN
+F 2 "keyboard_project:APTF1616SEJ3ZGGVBDC" H 7600 1450 50  0001 C CNN
 F 3 "~" H 7600 1450 50  0001 C CNN
 	1    7600 1500
