File: test_board/ledchain0.sch (KiCad schematic (older format))
At the start: 32 parts, among them U201 WS2811, U202 WS2811, U203 WS2811, U204 WS2811, U205 WS2811, U206 WS2811, U207 WS2811, U208 WS2811, U209 WS2811, U210 WS2811, U211 WS2811, U212 WS2811, U213 WS2811, U214 WS2811, U215 WS2811, U216 WS2811

Commit message: update schematic to CRGB LEDs and move footprints on pcb
Parts:
- D201, D202, D203, D204, D205, D206, D207, D208, D209, D210, D211, D212, D213, D214, D215, D216: value LED_RCBG -> LED_CRBG; symbol Device:LED_RCBG -> Device:LED_CRGB
Connections:
- net GND: now also D201.1 (K), D202.1 (K), D203.1 (K), D204.1 (K), D205.1 (K), D206.1 (K), D207.1 (K), D208.1 (K), D209.1 (K), D210.1 (K), D211.1 (K), D212.1 (K), D213.1 (K), D214.1 (K), D215.1 (K), D216.1 (K); no longer D201.2 (K), D202.2 (K), D203.2 (K), D204.2 (K), D205.2 (K), D206.2 (K), D207.2 (K), D208.2 (K), D209.2 (K), D210.2 (K), D211.2 (K), D212.2 (K), D213.2 (K), D214.2 (K), D215.2 (K), D216.2 (K)
- net at U205.1 (OUTR): now also D205.2 (RA); no longer D205.1 (RA)
- net at D205.3 (GA): now also U205.2 (OUTG); no longer U205.3 (OUTB)
- net at D205.4 (BA): now also U205.3 (OUTB); no longer U205.2 (OUTG)
- net at U204.1 (OUTR): now also D204.2 (RA); no longer D204.1 (RA)
- net at D204.3 (GA): now also U204.2 (OUTG); no longer U204.3 (OUTB)
- net at D204.4 (BA): now also U204.3 (OUTB); no longer U204.2 (OUTG)
- net at U203.1 (OUTR): now also D203.2 (RA); no longer D203.1 (RA)
- net at D203.3 (GA): now also U203.2 (OUTG); no longer U203.3 (OUTB)
- net at D203.4 (BA): now also U203.3 (OUTB); no longer U203.2 (OUTG)
- net at U202.1 (OUTR): now also D202.2 (RA); no longer D202.1 (RA)
- net at D202.3 (GA): now also U202.2 (OUTG); no longer U202.3 (OUTB)
- net at D202.4 (BA): now also U202.3 (OUTB); no longer U202.2 (OUTG)
- net at U201.1 (OUTR): now also D201.2 (RA); no longer D201.1 (RA)
- net at D201.3 (GA): now also U201.2 (OUTG); no longer U201.3 (OUTB)
- net at D201.4 (BA): now also U201.3 (OUTB); no longer U201.2 (OUTG)
- net at U210.1 (OUTR): now also D210.2 (RA); no longer D210.1 (RA)
- net at D210.3 (GA): now also U210.2 (OUTG); no longer U210.3 (OUTB)
- net at D210.4 (BA): now also U210.3 (OUTB); no longer U210.2 (OUTG)
- net at U209.1 (OUTR): now also D209.2 (RA); no longer D209.1 (RA)
- net at D209.3 (GA): now also U209.2 (OUTG); no longer U209.3 (OUTB)
- net at D209.4 (BA): now also U209.3 (OUTB); no longer U209.2 (OUTG)
- net at U208.1 (OUTR): now also D208.2 (RA); no longer D208.1 (RA)
- net at D208.3 (GA): now also U208.2 (OUTG); no longer U208.3 (OUTB)
- net at D208.4 (BA): now also U208.3 (OUTB); no longer U208.2 (OUTG)
- net at U207.1 (OUTR): now also D207.2 (RA); no longer D207.1 (RA)
- net at D207.3 (GA): now also U207.2 (OUTG); no longer U207.3 (OUTB)
- net at D207.4 (BA): now also U207.3 (OUTB); no longer U207.2 (OUTG)
- net at U206.1 (OUTR): now also D206.2 (RA); no longer D206.1 (RA)
- net at D206.3 (GA): now also U206.2 (OUTG); no longer U206.3 (OUTB)
- net at D206.4 (BA): now also U206.3 (OUTB); no longer U206.2 (OUTG)
- net at U215.1 (OUTR): now also D215.2 (RA); no longer D215.1 (RA)
- net at D215.3 (GA): now also U215.2 (OUTG); no longer U215.3 (OUTB)
- net at D215.4 (BA): now also U215.3 (OUTB); no longer U215.2 (OUTG)
- net at U214.1 (OUTR): now also D214.2 (RA); no longer D214.1 (RA)
- net at D214.3 (GA): now also U214.2 (OUTG); no longer U214.3 (OUTB)
- net at D214.4 (BA): now also U214.3 (OUTB); no longer U214.2 (OUTG)
- net at U213.1 (OUTR): now also D213.2 (RA); no longer D213.1 (RA)
- net at D213.3 (GA): now also U213.2 (OUTG); no longer U213.3 (OUTB)
- net at D213.4 (BA): now also U213.3 (OUTB); no longer U213.2 (OUTG)
- net at U212.1 (OUTR): now also D212.2 (RA); no longer D212.1 (RA)
- net at D212.3 (GA): now also U212.2 (OUTG); no longer U212.3 (OUTB)
- net at D212.4 (BA): now also U212.3 (OUTB); no longer U212.2 (OUTG)
- net at U211.1 (OUTR): now also D211.2 (RA); no longer D211.1 (RA)
- net at D211.3 (GA): now also U211.2 (OUTG); no longer U211.3 (OUTB)
- net at D211.4 (BA): now also U211.3 (OUTB); no longer U211.2 (OUTG)
- net at U216.1 (OUTR): now also D216.2 (RA); no longer D216.1 (RA)
- net at D216.3 (GA): now also U216.2 (OUTG); no longer U216.3 (OUTB)
- net at D216.4 (BA): now also U216.3 (OUTB); no longer U216.2 (OUTG)
Changed lines of the file:
@@
 	2650 6200 2650 6100
 $Comp
-L Device:LED_RCBG D?
+L Device:LED_CRGB D?
 U 1 1 5DE60084
 P 2950 6100
@@
 AR Path="/5DD36755/5DE60084" Ref="D205"  Part="1"
 F 0 "D205" H 2950 6597 50  0000 C CNN
-F 1 "LED_RCBG" H 2950 6506 50  0000 C CNN
+F 1 "LED_CRBG" H 2950 6506 50  0000 C CNN
 F 2 "keyboard_project:APTF1616SEJ3ZGGVBDC" H 2950 6050 50  0001 C CNN
 F 3 "~" H 2950 6050 50  0001 C CNN
@@
 	2650 5050 2650 4950
 $Comp
-L Device:LED_RCBG D?
+L Device:LED_CRGB D?
 U 1 1 5DE600AC
 P 2950 4950
@@
 AR Path="/5DD36755/5DE600AC" Ref="D204"  Part="1"
 F 0 "D204" H 2950 5447 50  0000 C CNN
-F 1 "LED_RCBG" H 2950 5356 50  0000 C CNN
+F 1 "LED_CRBG" H 2950 5356 50  0000 C CNN
 F 2 "keyboard_project:APTF1616SEJ3ZGGVBDC" H 2950 4900 50  0001 C CNN
 F 3 "~" H 2950 4900 50  0001 C CNN
@@
 	2650 3900 2650 3800
 $Comp
-L Device:LED_RCBG D?
+L Device:LED_CRGB D?
 U 1 1 5DE600D4
 P 2950 3800
@@
 AR Path="/5DD36755/5DE600D4" Ref="D203"  Part="1"
 F 0 "D203" H 2950 4297 50  0000 C CNN
-F 1 "LED_RCBG" H 2950 4206 50  0000 C CNN
+F 1 "LED_CRBG" H 2950 4206 50  0000 C CNN
 F 2 "keyboard_project:APTF1616SEJ3ZGGVBDC" H 2950 3750 50  0001 C CNN
 F 3 "~" H 2950 3750 50  0001 C CNN
@@
 	2650 2750 2650 2650
 $Comp
-L Device:LED_RCBG D?
+L Device:LED_CRGB D?
 U 1 1 5DE600FC
 P 2950 2650
@@
 AR Path="/5DD36755/5DE600FC" Ref="D202"  Part="1"
 F 0 "D202" H 2950 3147 50  0000 C CNN
-F 1 "LED_RCBG" H 2950 3056 50  0000 C CNN
+F 1 "LED_CRBG" H 2950 3056 50  0000 C CNN
 F 2 "keyboard_project:APTF1616SEJ3ZGGVBDC" H 2950 2600 50  0001 C CNN
 F 3 "~" H 2950 2600 50  0001 C CNN
@@
 	2650 1600 2650 1500
 $Comp
-L Device:LED_RCBG D?
+L Device:LED_CRGB D?
 U 1 1 5DE60123
 P 2950 1500
@@
 AR Path="/5DD36755/5DE60123" Ref="D201"  Part="1"
 F 0 "D201" H 2950 1997 50  0000 C CNN
-F 1 "LED_RCBG" H 2950 1906 50  0000 C CNN
+F 1 "LED_CRBG" H 2950 1906 50  0000 C CNN
 F 2 "keyboard_project:APTF1616SEJ3ZGGVBDC" H 2950 1450 50  0001 C CNN
 F 3 "~" H 2950 1450 50  0001 C CNN
@@
 	4200 6200 4200 6100
 $Comp
-L Device:LED_RCBG D?
+L Device:LED_CRGB D?
 U 1 1 5DE6015B
 P 4500 6100
@@
 AR Path="/5DD36755/5DE6015B" Ref="D210"  Part="1"
 F 0 "D210" H 4500 6597 50  0000 C CNN
-F 1 "LED_RCBG" H 4500 6506 50  0000 C CNN
+F 1 "LED_CRBG" H 4500 6506 50  0000 C CNN
 F 2 "keyboard_project:APTF1616SEJ3ZGGVBDC" H 4500 6050 50  0001 C CNN
 F 3 "~" H 4500 6050 50  0001 C CNN
@@
 	4200 5050 4200 4950
 $Comp
-L Device:LED_RCBG D?
+L Device:LED_CRGB D?
 U 1 1 5DE60183
 P 4500 4950
@@
 AR Path="/5DD36755/5DE60183" Ref="D209"  Part="1"
 F 0 "D209" H 4500 5447 50  0000 C CNN
-F 1 "LED_RCBG" H 4500 5356 50  0000 C CNN
+F 1 "LED_CRBG" H 4500 5356 50  0000 C CNN
 F 2 "keyboard_project:APTF1616SEJ3ZGGVBDC" H 4500 4900 50  0001 C CNN
 F 3 "~" H 4500 4900 50  0001 C CNN
@@
 	4200 3900 4200 3800
 $Comp
-L Device:LED_RCBG D?
+L Device:LED_CRGB D?
 U 1 1 5DE601AB
 P 4500 3800
@@
 AR Path="/5DD36755/5DE601AB" Ref="D208"  Part="1"
 F 0 "D208" H 4500 4297 50  0000 C CNN
-F 1 "LED_RCBG" H 4500 4206 50  0000 C CNN
+F 1 "LED_CRBG" H 4500 4206 50  0000 C CNN
 F 2 "keyboard_project:APTF1616SEJ3ZGGVBDC" H 4500 3750 50  0001 C CNN
 F 3 "~" H 4500 3750 50  0001 C CNN
@@
 	4200 2750 4200 2650
 $Comp
-L Device:LED_RCBG D?
+L Device:LED_CRGB D?
 U 1 1 5DE601D3
 P 4500 2650
@@
 AR Path="/5DD36755/5DE601D3" Ref="D207"  Part="1"
 F 0 "D207" H 4500 3147 50  0000 C CNN
-F 1 "LED_RCBG" H 4500 3056 50  0000 C CNN
+F 1 "LED_CRBG" H 4500 3056 50  0000 C CNN
 F 2 "keyboard_project:APTF1616SEJ3ZGGVBDC" H 4500 2600 50  0001 C CNN
 F 3 "~" H 4500 2600 50  0001 C CNN
@@
 	4200 1600 4200 1500
 $Comp
-L Device:LED_RCBG D?
+L Device:LED_CRGB D?
 U 1 1 5DE601FA
 P 4500 1500
@@
 AR Path="/5DD36755/5DE601FA" Ref="D206"  Part="1"
 F 0 "D206" H 4500 1997 50  0000 C CNN
-F 1 "LED_RCBG" H 4500 1906 50  0000 C CNN
+F 1 "LED_CRBG" H 4500 1906 50  0000 C CNN
 F 2 "keyboard_project:APTF1616SEJ3ZGGVBDC" H 4500 1450 50  0001 C CNN
 F 3 "~" H 4500 1450 50  0001 C CNN
@@
 	5750 6200 5750 6100
 $Comp
-L Device:LED_RCBG D?
+L Device:LED_CRGB D?
 U 1 1 5DE60233
 P 6050 6100
@@
 AR Path="/5DD36755/5DE60233" Ref="D215"  Part="1"
 F 0 "D215" H 6050 6597 50  0000 C CNN
-F 1 "LED_RCBG" H 6050 6506 50  0000 C CNN
+F 1 "LED_CRBG" H 6050 6506 50  0000 C CNN
 F 2 "keyboard_project:APTF1616SEJ3ZGGVBDC" H 6050 6050 50  0001 C CNN
 F 3 "~" H 6050 6050 50  0001 C CNN
@@
 	5750 5050 5750 4950
 $Comp
-L Device:LED_RCBG D?
+L Device:LED_CRGB D?
 U 1 1 5DE6025B
 P 6050 4950
@@
 AR Path="/5DD36755/5DE6025B" Ref="D214"  Part="1"
 F 0 "D214" H 6050 5447 50  0000 C CNN
-F 1 "LED_RCBG" H 6050 5356 50  0000 C CNN
+F 1 "LED_CRBG" H 6050 5356 50  0000 C CNN
 F 2 "keyboard_project:APTF1616SEJ3ZGGVBDC" H 6050 4900 50  0001 C CNN
 F 3 "~" H 6050 4900 50  0001 C CNN
@@
 	5750 3900 5750 3800
 $Comp
-L Device:LED_RCBG D?
+L Device:LED_CRGB D?
 U 1 1 5DE60283
 P 6050 3800
@@
 AR Path="/5DD36755/5DE60283" Ref="D213"  Part="1"
 F 0 "D213" H 6050 4297 50  0000 C CNN
-F 1 "LED_RCBG" H 6050 4206 50  0000 C CNN
+F 1 "LED_CRBG" H 6050 4206 50  0000 C CNN
 F 2 "keyboard_project:APTF1616SEJ3ZGGVBDC" H 6050 3750 50  0001 C CNN
 F 3 "~" H 6050 3750 50  0001 C CNN
@@
 	5750 2750 5750 2650
 $Comp
-L Device:LED_RCBG D?
+L Device:LED_CRGB D?
 U 1 1 5DE602AB
 P 6050 2650
@@
 AR Path="/5DD36755/5DE602AB" Ref="D212"  Part="1"
 F 0 "D212" H 6050 3147 50  0000 C CNN
-F 1 "LED_RCBG" H 6050 3056 50  0000 C CNN
+F 1 "LED_CRBG" H 6050 3056 50  0000 C CNN
 F 2 "keyboard_project:APTF1616SEJ3ZGGVBDC" H 6050 2600 50  0001 C CNN
 F 3 "~" H 6050 2600 50  0001 C CNN
@@
 	5750 1600 5750 1500
 $Comp
-L Device:LED_RCBG D?
+L Device:LED_CRGB D?
 U 1 1 5DE602D2
 P 6050 1500
@@
 AR Path="/5DD36755/5DE602D2" Ref="D211"  Part="1"
 F 0 "D211" H 6050 1997 50  0000 C CNN
-F 1 "LED_RCBG" H 6050 1906 50  0000 C CNN
+F 1 "LED_CRBG" H 6050 1906 50  0000 C CNN
 F 2 "keyboard_project:APTF1616SEJ3ZGGVBDC" H 6050 1450 50  0001 C CNN
 F 3 "~" H 6050 1450 50  0001 C CNN
@@
 	7300 1600 7300 1500
 $Comp
-L Device:LED_RCBG D?
+L Device:LED_CRGB D?
 U 1 1 5DE603A6
 P 7600 1500
@@
 AR Path="/5DD36755/5DE603A6" Ref="D216"  Part="1"
 F 0 "D216" H 7600 1997 50  0000 C CNN
-F 1 "LED_RCBG" H 7600 1906 50  0000 C CNN
+F 1 "LED_CRBG" H 7600 1906 50  0000 C CNN
 F 2 "keyboard_project:APTF1616SEJ3ZGGVBDC" H 7600 1450 50  0001 C CNN
 F 3 "~" H 7600 1450 50  0001 C CNN
