File: test_board/Keymatrix.sch (KiCad schematic (older format))
At the start: 32 parts, among them K301 KEYSW, K302 KEYSW, K303 KEYSW, K304 KEYSW, K305 KEYSW, K306 KEYSW, K307 KEYSW, K308 KEYSW, K309 KEYSW, K310 KEYSW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

Commit message: update schematic to smd diode
Parts:
- D301, D302, D303, D304, D305, D306, D307, D308, D309, D310, D311, D312, D313, D314, D315, D316: footprint keyboard_parts:D_axial -> Diode_SMD:D_SOD-523
Changed lines of the file:
@@
 F 0 "D301" H 4122 3300 60  0000 R CNN
 F 1 "D" V 4400 3300 60  0001 C CNN
-F 2 "keyboard_parts:D_axial" H 4250 3350 60  0001 C CNN
+F 2 "Diode_SMD:D_SOD-523" H 4250 3350 60  0001 C CNN
 F 3 "" H 4250 3350 60  0000 C CNN
 	1    4250 3350
@@
 F 0 "D302" H 4122 3800 60  0000 R CNN
 F 1 "D" V 4400 3800 60  0001 C CNN
-F 2 "keyboard_parts:D_axial" H 4250 3850 60  0001 C CNN
+F 2 "Diode_SMD:D_SOD-523" H 4250 3850 60  0001 C CNN
 F 3 "" H 4250 3850 60  0000 C CNN
 	1    4250 3850
@@
 F 0 "D303" H 4122 4300 60  0000 R CNN
 F 1 "D" V 4400 4300 60  0001 C CNN
-F 2 "keyboard_parts:D_axial" H 4250 4350 60  0001 C CNN
+F 2 "Diode_SMD:D_SOD-523" H 4250 4350 60  0001 C CNN
 F 3 "" H 4250 4350 60  0000 C CNN
 	1    4250 4350
@@
 F 0 "D304" H 4122 4800 60  0000 R CNN
 F 1 "D" V 4400 4800 60  0001 C CNN
-F 2 "keyboard_parts:D_axial" H 4250 4850 60  0001 C CNN
+F 2 "Diode_SMD:D_SOD-523" H 4250 4850 60  0001 C CNN
 F 3 "" H 4250 4850 60  0000 C CNN
 	1    4250 4850
@@
 F 0 "D305" H 4972 3300 60  0000 R CNN
 F 1 "D" V 5250 3300 60  0001 C CNN
-F 2 "keyboard_parts:D_axial" H 5100 3350 60  0001 C CNN
+F 2 "Diode_SMD:D_SOD-523" H 5100 3350 60  0001 C CNN
 F 3 "" H 5100 3350 60  0000 C CNN
 	1    5100 3350
@@
 F 0 "D306" H 4972 3800 60  0000 R CNN
 F 1 "D" V 5250 3800 60  0001 C CNN
-F 2 "keyboard_parts:D_axial" H 5100 3850 60  0001 C CNN
+F 2 "Diode_SMD:D_SOD-523" H 5100 3850 60  0001 C CNN
 F 3 "" H 5100 3850 60  0000 C CNN
 	1    5100 3850
@@
 F 0 "D307" H 4972 4300 60  0000 R CNN
 F 1 "D" V 5250 4300 60  0001 C CNN
-F 2 "keyboard_parts:D_axial" H 5100 4350 60  0001 C CNN
+F 2 "Diode_SMD:D_SOD-523" H 5100 4350 60  0001 C CNN
 F 3 "" H 5100 4350 60  0000 C CNN
 	1    5100 4350
@@
 F 0 "D308" H 4972 4800 60  0000 R CNN
 F 1 "D" V 5250 4800 60  0001 C CNN
-F 2 "keyboard_parts:D_axial" H 5100 4850 60  0001 C CNN
+F 2 "Diode_SMD:D_SOD-523" H 5100 4850 60  0001 C CNN
 F 3 "" H 5100 4850 60  0000 C CNN
 	1    5100 4850
@@
 F 0 "D309" H 5822 3300 60  0000 R CNN
 F 1 "D" V 6100 3300 60  0001 C CNN
-F 2 "keyboard_parts:D_axial" H 5950 3350 60  0001 C CNN
+F 2 "Diode_SMD:D_SOD-523" H 5950 3350 60  0001 C CNN
 F 3 "" H 5950 3350 60  0000 C CNN
 	1    5950 3350
@@
 F 0 "D310" H 5822 3800 60  0000 R CNN
 F 1 "D" V 6100 3800 60  0001 C CNN
-F 2 "keyboard_parts:D_axial" H 5950 3850 60  0001 C CNN
+F 2 "Diode_SMD:D_SOD-523" H 5950 3850 60  0001 C CNN
 F 3 "" H 5950 3850 60  0000 C CNN
 	1    5950 3850
@@
 F 0 "D311" H 5822 4300 60  0000 R CNN
 F 1 "D" V 6100 4300 60  0001 C CNN
-F 2 "keyboard_parts:D_axial" H 5950 4350 60  0001 C CNN
+F 2 "Diode_SMD:D_SOD-523" H 5950 4350 60  0001 C CNN
 F 3 "" H 5950 4350 60  0000 C CNN
 	1    5950 4350
@@
 F 0 "D312" H 5822 4800 60  0000 R CNN
 F 1 "D" V 6100 4800 60  0001 C CNN
-F 2 "keyboard_parts:D_axial" H 5950 4850 60  0001 C CNN
+F 2 "Diode_SMD:D_SOD-523" H 5950 4850 60  0001 C CNN
 F 3 "" H 5950 4850 60  0000 C CNN
 	1    5950 4850
@@
 F 0 "D313" H 6672 3300 60  0000 R CNN
 F 1 "D" V 6950 3300 60  0001 C CNN
-F 2 "keyboard_parts:D_axial" H 6800 3350 60  0001 C CNN
+F 2 "Diode_SMD:D_SOD-523" H 6800 3350 60  0001 C CNN
 F 3 "" H 6800 3350 60  0000 C CNN
 	1    6800 3350
@@
 F 0 "D314" H 6672 3800 60  0000 R CNN
 F 1 "D" V 6950 3800 60  0001 C CNN
-F 2 "keyboard_parts:D_axial" H 6800 3850 60  0001 C CNN
+F 2 "Diode_SMD:D_SOD-523" H 6800 3850 60  0001 C CNN
 F 3 "" H 6800 3850 60  0000 C CNN
 	1    6800 3850
@@
 F 0 "D315" H 6672 4300 60  0000 R CNN
 F 1 "D" V 6950 4300 60  0001 C CNN
-F 2 "keyboard_parts:D_axial" H 6800 4350 60  0001 C CNN
+F 2 "Diode_SMD:D_SOD-523" H 6800 4350 60  0001 C CNN
 F 3 "" H 6800 4350 60  0000 C CNN
 	1    6800 4350
@@
 F 0 "D316" H 6672 4800 60  0000 R CNN
 F 1 "D" V 6950 4800 60  0001 C CNN
-F 2 "keyboard_parts:D_axial" H 6800 4850 60  0001 C CNN
+F 2 "Diode_SMD:D_SOD-523" H 6800 4850 60  0001 C CNN
 F 3 "" H 6800 4850 60  0000 C CNN
 	1    6800 4850
